Commit message: floor added + minimal and test URDF

File: install/ur5e_description/share/ur5e_description/urdf/ur5e.urdf.xacro (robot description, xacro)
@@ -1 +1 @@
-/home/arya/ROS/UR5e/src/ur5e_description/urdf/ur5e.urdf.xacro
+/home/ah66586/ros2_ws/UR5e_3DP/src/ur5e_description/urdf/ur5e.urdf.xacro

File: src/ur5e_description/urdf/ur5e.urdf.xacro (robot description, xacro)
@@ -1,7 +1,5 @@
 <?xml version="1.0"?>
 <robot xmlns:xacro="http://www.ros.org/wiki/xacro" name="ur5e">
-  <!-- Import UR5e macro from ur_description -->
   <xacro:include filename="$(find ur_description)/urdf/ur_macro.xacro"/>
-  <!-- Instantiate the robot -->
   <xacro:arg name="name" default="ur"/>
   <xacro:arg name="ur_type" default="ur5e"/>
@@ -20,6 +18,25 @@
     <origin xyz="0 0 0" rpy="0 0 0" />
   </xacro:ur_robot>
-  <!-- World link -->
   <link name="world" />
+  <link name="floor">
+    <visual>
+      <geometry>
+        <box size="3.048 3.048 0.0254"/>
+      </geometry>
+      <material name="floor_color">
+        <color rgba="0.3 0.3 0.3 1"/>
+      </material>
+    </visual>
+    <collision>
+      <geometry>
+        <box size="3.048 3.048 0.0254"/>
+      </geometry>
+    </collision>
+  </link>
+  <joint name="world_to_floor" type="fixed">
+    <parent link="world"/>
+    <child link="floor"/>
+    <origin xyz="0 0 -0.0127" rpy="0 0 0"/>
+  </joint>
   <link name="tool_head">
     <visual>
@@ -31,7 +48,11 @@
       </material>
     </visual>
+    <collision>
+      <origin xyz="0 -0.09 0" rpy="0 0 0"/>
+      <geometry>
+        <box size="0.15 0.21 0.15"/>
+      </geometry>
+    </collision>
   </link>
-  <!-- Attach tool head to wrist_3_link (which is named 'wrist_3_link' in the macro) -->
-  <!-- Note: The macro typically prefixes link names if tf_prefix is set, but here it is empty -->
   <joint name="tool_head_joint" type="fixed">
     <parent link="tool0"/>
@@ -39,5 +60,4 @@
     <origin xyz="0 0 0" rpy="0 0 0"/>
   </joint>
-  <!-- Tool Tip (TCP) Link -->
   <link name="tool_tip">
     <visual>
